File: MyZON-X.kicad_sch (KiCad schematic)
At the start: 20 parts, among them CON1 EDG-CON-ZX81, J2 Conn_02x03_Counter_Clockwise, U1 AY-3-8910, U2. 74HCT74, U3. 74HCT08, U4 74HCT11, U4. 74HCT11, U5. 74HCT02

Commit message: commit 2
Other:
- title: JonZON-Xa -> JonZON-X
Changed lines of the file:
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@@
 	(paper "A4")
 	(title_block
-		(title "JonZON-Xa")
+		(title "JonZON-X")
 		(date "2025-08-01")
 		(rev "1.0")

Commit message: change 1
Other:
- title: JonZON-X -> JonZON-Xa
Changed lines of the file:
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@@
 	(paper "A4")
 	(title_block
-		(title "JonZON-X")
+		(title "JonZON-Xa")
 		(date "2025-08-01")
 		(rev "1.0")
