File: JONZON-X-81.kicad_pcb (KiCad board)
At the start: 2 copper layers, 63.5 x 101 mm, 30 parts, among them SW1 SW_DIP_x03, U1 AY-3-8910, U2 74HCT74, U3 74HCT08, U4 74HCT11, U5 74HCT02

Commit message: 1.2
Connections:
- R4 pad 1: /OUTB -> /OUTC
- R6 pad 2: /OUTC -> /OUTB
- R7 pad 2: /OUTC -> /OUTB
Routing:
- net /OUTB: track 5.34 -> 19.1 mm
- net /OUTC: track 29.9 -> 22.5 mm
- net Net-(CO3-Pin_1): track 59.8 -> 58.7 mm, vias 1 -> 0
- net GND_AUDIO: vias 316 -> 328
- net GND: vias 361 -> 362
Other:
- board text added: "JONZON-X-81 Rev: 1.2 2025 - J.Gratton"
- board text added: "Rev: 1.2 set Channel A Left (tip), Channel C Right (sleeve) and Chabbel B Mixed."
- board text removed: "JONZON-X-81 Rev: 1.1 2025 - J.Gratton"
Changed lines of the file:
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@@
 		(title "JONZON-X-81")
 		(date "2025-08-11")
-		(rev "1.1")
+		(rev "1.2")
 	)
 	(layers
@@
 			(layers "*.Cu" "*.Mask")
 			(remove_unused_layers no)
-			(net 51 "/OUTB")
+			(net 53 "/OUTC")
 			(pintype "passive")
 		)
@@
 			(layers "*.Cu" "*.Mask")
 			(remove_unused_layers no)
-			(net 53 "/OUTC")
+			(net 51 "/OUTB")
 			(pintype "passive")
 		)
@@
 			(layers "*.Cu" "*.Mask")
 			(remove_unused_layers no)
-			(net 53 "/OUTC")
+			(net 51 "/OUTB")
 			(pintype "passive")
 		)
@@
 		(layer "Edge.Cuts")
 	)
+	(gr_text "Rev: 1.2 set Channel A Left (tip), Channel C Right (sleeve) and Chabbel B Mixed."
+		(at 177.8 174.625 0)
+		(layer "F.Cu")
+		(effects
+			(font
+				(size 1 1)
+				(thickness 0.2)
+			)
+			(justify left bottom)
+		)
+	)
 	(gr_text "Rev: 1.1 was a change to the Audio Jack connections.\nLeft and Right where connected to Shunts A and B.\nThis also resulted in a Left and Right swap, so Channel A and B where reveresed to compensate."
 		(at 177.8 171.45 0)
@@
 		)
 	)
-	(gr_text "JONZON-X-81 Rev: 1.1\n2025 - J.Gratton"
+	(gr_text "JONZON-X-81 Rev: 1.2\n2025 - J.Gratton"
 		(at 54.61 131.445 0)
 		(layer "F.SilkS")
@@
 	)
 	(via
-		(at 103.505 86.995)
-		(size 0.6)
-		(drill 0.3)
-		(layers "F.Cu" "B.Cu")
-		(free yes)
-		(net 5)
-	)
-	(via
 		(at 81.915 123.825)
 		(size 0.6)
@@
 	)
 	(via
-		(at 102.235 86.995)
-		(size 0.6)
-		(drill 0.3)
-		(layers "F.Cu" "B.Cu")
-		(free yes)
-		(net 5)
-	)
-	(via
 		(at 110.49 96.52)
 		(size 0.6)
@@
 	)
 	(via
+		(at 100.33 86.995)
+		(size 0.6)
+		(drill 0.3)
+		(layers "F.Cu" "B.Cu")
+		(free yes)
+		(net 5)
+	)
+	(via
 		(at 57.15 134.62)
 		(size 0.6)
@@
 	)
 	(via
+		(at 99.06 86.995)
+		(size 0.6)
+		(drill 0.3)
+		(layers "F.Cu" "B.Cu")
+		(free yes)
+		(net 5)
+	)
+	(via
 		(at 91.44 86.995)
 		(size 0.6)
@@
 	)
 	(via
+		(at 101.6 86.995)
+		(size 0.6)
+		(drill 0.3)
+		(layers "F.Cu" "B.Cu")
+		(free yes)
+		(net 5)
+	)
+	(via
 		(at 53.34 119.38)
 		(size 0.6)
@@
 	)
 	(segment
-		(start 76.5768 61.2182)
-		(end 76.5768 55.4557)
+		(start 79.375 54.61)
+		(end 86.355 54.61)
 		(width 0.2)
 		(layer "F.Cu")
@@
 	)
 	(segment
-		(start 101.8451 57.84)
-		(end 104.14 60.1349)
+		(start 76.5768 57.4082)
+		(end 79.375 54.61)
 		(width 0.2)
 		(layer "F.Cu")
@@
 	)
 	(segment
-		(start 104.14 67.29)
-		(end 106.065 69.215)
+		(start 101.8451 57.84)
+		(end 104.14 60.1349)
 		(width 0.2)
 		(layer "F.Cu")
@@
 	)
 	(segment
-		(start 66.675 71.12)
-		(end 76.5768 61.2182)
+		(start 76.5768 61.2182)
+		(end 76.5768 57.4082)
 		(width 0.2)
 		(layer "F.Cu")
@@
 	)
 	(segment
-		(start 104.14 60.1349)
-		(end 104.14 67.29)
+		(start 104.14 67.29)
+		(end 106.065 69.215)
 		(width 0.2)
 		(layer "F.Cu")
 		(net 12)
 	)
-	(via
-		(at 76.5768 55.4557)
-		(size 0.6)
-		(drill 0.3)
-		(layers "F.Cu" "B.Cu")
-		(net 12)
-	)
 	(segment
-		(start 86.995 54.61)
-		(end 89.0415 56.6565)
+		(start 104.14 60.1349)
+		(end 104.14 67.29)
 		(width 0.2)
-		(layer "B.Cu")
+		(layer "F.Cu")
 		(net 12)
 	)
 	(segment
-		(start 86.355 54.61)
-		(end 85.2033 54.61)
+		(start 66.675 71.12)
+		(end 76.5768 61.2182)
 		(width 0.2)
-		(layer "B.Cu")
+		(layer "F.Cu")
 		(net 12)
 	)
 	(segment
-		(start 84.3576 55.4557)
-		(end 85.2033 54.61)
+		(start 86.995 54.61)
+		(end 89.0415 56.6565)
 		(width 0.2)
 		(layer "B.Cu")
@@
 	)
 	(segment
-		(start 76.5768 55.4557)
-		(end 84.3576 55.4557)
-		(width 0.2)
-		(layer "B.Cu")
-		(net 12)
-	)
-	(segment
 		(start 106.675 144.78)
 		(end 106.675 133.355)
@@
 	)
 	(segment
-		(start 102.235 71.12)
-		(end 102.86 71.745)
+		(start 93.98 71.12)
+		(end 92.075 71.12)
+		(width 0.2)
+		(layer "B.Cu")
+		(net 51)
+	)
+	(segment
+		(start 95.885 73.025)
+		(end 93.98 71.12)
 		(width 0.2)
 		(layer "B.Cu")
@@
 	(segment
 		(start 102.86 76.2)
-		(end 102.86 71.745)
+		(end 102.86 74.285)
+		(width 0.2)
+		(layer "B.Cu")
+		(net 51)
+	)
+	(segment
+		(start 102.86 74.285)
+		(end 101.6 73.025)
+		(width 0.2)
+		(layer "B.Cu")
+		(net 51)
+	)
+	(segment
+		(start 101.6 73.025)
+		(end 95.885 73.025)
+		(width 0.2)
+		(layer "B.Cu")
+		(net 51)
+	)
+	(segment
+		(start 92.075 71.12)
+		(end 86.995 71.12)
 		(width 0.2)
 		(layer "B.Cu")
@@
 	)
 	(segment
-		(start 102.86 89.9383)
-		(end 93.97 81.0483)
+		(start 104.14 84.455)
+		(end 102.854 85.741)
 		(width 0.2)
 		(layer "F.Cu")
@@
 	)
 	(segment
-		(start 93.97 81.0483)
-		(end 93.97 73.015)
+		(start 102.854 85.741)
+		(end 102.854 91.434)
 		(width 0.2)
 		(layer "F.Cu")
@@
 	)
 	(segment
-		(start 102.86 91.44)
-		(end 102.86 89.9383)
+		(start 102.854 91.434)
+		(end 102.86 91.44)
 		(width 0.2)
 		(layer "F.Cu")
@@
 	)
 	(segment
-		(start 93.97 73.015)
-		(end 92.075 71.12)
+		(start 102.235 71.12)
+		(end 104.14 73.025)
 		(width 0.2)
 		(layer "F.Cu")
@@
 	)
 	(segment
-		(start 92.075 71.12)
-		(end 86.995 71.12)
+		(start 104.14 73.025)
+		(end 104.14 84.455)
+		(width 0.2)
+		(layer "F.Cu")
+		(net 53)
+	)
+	(segment
+		(start 102.235 71.12)
+		(end 102.86 71.745)
 		(width 0.2)
 		(layer "B.Cu")
@@
 	)
 	(via
+		(at 93.98 80.645)
+		(size 0.6)
+		(drill 0.3)
+		(layers "F.Cu" "B.Cu")
+		(free yes)
+		(net 93)
+	)
+	(via
 		(at 82.55 61.595)
 		(size 0.6)
@@
 	)
 	(via
+		(at 100.33 80.645)
+		(size 0.6)
+		(drill 0.3)
+		(layers "F.Cu" "B.Cu")
+		(free yes)
+		(net 93)
+	)
+	(via
 		(at 96.52 49.53)
 		(size 0.6)
@@
 	)
 	(via
+		(at 102.87 80.645)
+		(size 0.6)
+		(drill 0.3)
+		(layers "F.Cu" "B.Cu")
+		(free yes)
+		(net 93)
+	)
+	(via
 		(at 81.28 80.645)
 		(size 0.6)
@@
 	)
 	(via
+		(at 97.79 80.645)
+		(size 0.6)
+		(drill 0.3)
+		(layers "F.Cu" "B.Cu")
+		(free yes)
+		(net 93)
+	)
+	(via
 		(at 114.3 79.375)
 		(size 0.6)
@@
 	)
 	(via
+		(at 82.55 56.515)
+		(size 0.6)
+		(drill 0.3)
+		(layers "F.Cu" "B.Cu")
+		(free yes)
+		(net 93)
+	)
+	(via
 		(at 58.42 55.88)
 		(size 0.6)
@@
 	)
 	(via
+		(at 80.01 56.515)
+		(size 0.6)
+		(drill 0.3)
+		(layers "F.Cu" "B.Cu")
+		(free yes)
+		(net 93)
+	)
+	(via
 		(at 59.69 62.23)
 		(size 0.6)
@@
 	)
 	(via
+		(at 96.52 80.645)
+		(size 0.6)
+		(drill 0.3)
+		(layers "F.Cu" "B.Cu")
+		(free yes)
+		(net 93)
+	)
+	(via
 		(at 53.34 69.85)
 		(size 0.6)
@@
 	)
 	(via
+		(at 95.25 80.645)
+		(size 0.6)
+		(drill 0.3)
+		(layers "F.Cu" "B.Cu")
+		(free yes)
+		(net 93)
+	)
+	(via
 		(at 93.98 54.61)
 		(size 0.6)
@@
 	)
 	(via
+		(at 83.82 56.515)
+		(size 0.6)
+		(drill 0.3)
+		(layers "F.Cu" "B.Cu")
+		(free yes)
+		(net 93)
+	)
+	(via
 		(at 114.3 80.645)
 		(size 0.6)
@@
 	)
 	(via
+		(at 81.28 56.515)
+		(size 0.6)
+		(drill 0.3)
+		(layers "F.Cu" "B.Cu")
+		(free yes)
+		(net 93)
+	)
+	(via
 		(at 113.03 80.645)
 		(size 0.6)
@@
 	)
 	(via
+		(at 99.06 80.645)
+		(size 0.6)
+		(drill 0.3)
+		(layers "F.Cu" "B.Cu")
+		(free yes)
+		(net 93)
+	)
+	(via
 		(at 55.88 62.23)
 		(size 0.6)
@@
 	)
 	(via
+		(at 101.6 80.645)
+		(size 0.6)
+		(drill 0.3)
+		(layers "F.Cu" "B.Cu")
+		(free yes)
+		(net 93)
+	)
+	(via
 		(at 92.71 59.055)
 		(size 0.6)
@@
 		)
 	)
-	(group ""
-		(members "17594fdc-202c-4f89-92de-1fe9c80c4429" "783708c0-1574-46b5-9b98-afb5aa4aeeea"
-			"920e1c2b-d4b5-42d1-970a-63cfbfba0767" "abf504e9-643f-4472-b606-7263c096813d"
-			"b7988163-c927-44e3-b155-7ee1bc303cbe" "ba3feab8-825e-45c2-bfd6-a01a4fe87caf"
-			"fcc1b5f5-9fc1-4a71-8e26-35bde2b49357"
-		)
-	)
