File: JONZON-X-81.kicad_pcb (KiCad board)
At the start: 2 copper layers, 63.5 x 101 mm, 20 parts, among them SW1 SW_DIP_x01, U1 AY-3-8912, U2 74HCT74, U3 74HCT02, U4 74HCT11

Commit message: rev 1.3
Parts:
- added C7: 100nf, Capacitor_THT:C_Disc_D3.0mm_W1.6mm_P2.50mm, F.Cu at (90.8, 99.7)
- added C8: 100nf, Capacitor_THT:C_Disc_D3.0mm_W1.6mm_P2.50mm, F.Cu at (109.2, 99.7)
- added C9: 100nf, Capacitor_THT:C_Disc_D3.0mm_W1.6mm_P2.50mm, F.Cu at (111.1, 88.9)
- added CO3: THROUGH, Connector_PinHeader_2.54mm:PinHeader_1x03_P2.54mm_Vertical, F.Cu at (86.4, 54.6)
- added R10: 100R, Resistor_THT:R_Axial_DIN0207_L6.3mm_D2.5mm_P7.62mm_Horizontal, F.Cu at (71.8, 63.5)
- added R11: 100R, Resistor_THT:R_Axial_DIN0207_L6.3mm_D2.5mm_P7.62mm_Horizontal, F.Cu at (66.7, 63.5)
- added R12: 0R, Resistor_THT:R_Axial_DIN0207_L6.3mm_D2.5mm_P7.62mm_Horizontal, F.Cu at (55.2, 87.6)
- added R8: 390R, Resistor_THT:R_Axial_DIN0207_L6.3mm_D2.5mm_P7.62mm_Horizontal, F.Cu at (81.9, 63.5)
- added R9: 390R, Resistor_THT:R_Axial_DIN0207_L6.3mm_D2.5mm_P7.62mm_Horizontal, F.Cu at (76.8, 63.5)
- added U5: 74HCT02, Package_DIP:DIP-14_W7.62mm_Socket_LongPads, F.Cu at (104.2, 104.1)
- R1: value 10K -> 47K
- R2: value 390R -> 47K
- R3: value 820R -> 47K
- R4: value 820R -> 390R
- R6, R7: value 390R -> 820R
- SW1: value SW_DIP_x01 -> SW_DIP_x03; footprint Button_Switch_SMD:SW_DIP_SPSTx01_Slide_9.78x4.72mm_W8.61mm_P2.54mm -> Button_Switch_THT:SW_DIP_SPSTx03_Slide_9.78x9.8mm_W7.62mm_P2.54mm
- U1: value AY-3-8912 -> AY-3-8910; footprint AY-3-8912:AY-3-8912 -> Package_DIP:DIP-40_W15.24mm_LongPads
- U3: value 74HCT02 -> 74HCT08
- moved CO1 123.0 mm to (85.1, 144.8)
- moved U4 79.3 mm to (88.3, 104.1)
- moved U2 79.2 mm to (55.9, 104.1)
- moved U3 78.4 mm to (71.8, 104.1)
- moved C5 66.2 mm to (58.4, 99.7)
- moved R2 63.3 mm to (92.7, 125.7), turned to -90 degrees
- moved R3 59.5 mm to (87.6, 125.7), turned to -90 degrees
- moved C6 52.1 mm to (74.3, 99.7)
- moved C3 47.4 mm to (106.1, 65.4)
- moved C4 46.8 mm to (106.1, 69.2)
- moved R1 39.3 mm to (97.8, 125.7), turned to -90 degrees
- moved SW1 34.5 mm to (109.2, 125.7), turned to -90 degrees
- moved R4 31.1 mm to (102.2, 71.1)
- moved U1 28.7 mm to (107.9, 76.2)
- moved R5 22.0 mm to (97.2, 71.1)
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Connections:
- C3 pad 1: VCC -> Net-(CO3-Pin_2)
- C3 pad 2: GND -> GND_AUDIO
- C4 pad 1: VCC -> Net-(CO3-Pin_1)
- C4 pad 2: GND -> GND_AUDIO
- CO1 pad A22: unconnected-(CO1-A6-PadA22) -> /A6
- CO1 pad A23: unconnected-(CO1-A5-PadA23) -> /A5
- CO1 pad B18: unconnected-(CO1-~{RD}-PadB18) -> /~{RD}
- CO2 pad 1: Net-(C1-Pad2) -> Net-(CO3-Pin_2)
- CO2 pad 4: Net-(C2-Pad2) -> Net-(CO3-Pin_1)
- CO2 pad 5: GND -> GND_AUDIO
- R2 pad 1: /OUTC -> VCC
- R2 pad 2: Net-(C1-Pad1) -> Net-(R2-Pad2)
- R3 pad 1: Net-(C1-Pad1) -> VCC
- R3 pad 2: /OUTB -> Net-(R3-Pad2)
- R4 pad 1: Net-(C2-Pad1) -> /OUTC
- R4 pad 2: /OUTB -> Net-(C1-Pad1)
- R6 pad 1: Net-(C1-Pad1) -> Net-(C2-Pad1)
- R6 pad 2: GND -> /OUTB
- R7 pad 1: Net-(C2-Pad1) -> Net-(C1-Pad1)
- R7 pad 2: GND -> /OUTB
- SW1 pad 1: /A4 -> Net-(R3-Pad2)
- SW1 pad 2: Net-(R1-Pad2) -> Net-(R2-Pad2)
- U1 pad 1: /OUTC -> GND
- U1 pad 15: /PSGCLK -> unconnected-(U1-IOA6-Pad15)
- U1 pad 16: /~{RESET} -> unconnected-(U1-IOA5-Pad16)
- U1 pad 17: VCC -> unconnected-(U1-IOA4-Pad17)
- U1 pad 18: /BDIR -> unconnected-(U1-IOA3-Pad18)
- U1 pad 19: VCC -> unconnected-(U1-IOA2-Pad19)
- U1 pad 20: /BC1 -> unconnected-(U1-IOA1-Pad20)
- U1 pad 21: /D7 -> unconnected-(U1-IOA0-Pad21)
- U1 pad 22: /D6 -> /PSGCLK
- U1 pad 23: /D5 -> /~{RESET}
- U1 pad 24: /D4 -> GND
- U1 pad 25: /D3 -> VCC
- U1 pad 26: /D2 -> unconnected-(U1-TEST2-Pad26)
- U1 pad 27: /D1 -> /BDIR
- U1 pad 28: /D0 -> VCC
- U1 pad 3: VCC -> /OUTB
- U1 pad 4: /OUTB -> /OUTA
- U1 pad 5: /OUTA -> unconnected-(U1-NC5-Pad5)
- U1 pad 6: GND -> unconnected-(U1-IOB7-Pad6)
- U3 pad 1: Net-(U3-Pad1) -> /VALID
- U3 pad 10: /BC1 -> GND
- U3 pad 11: /BDIR -> Net-(U3-Pad11)
- U3 pad 12: /BDIR -> /VALID
- U3 pad 13: Net-(U3-Pad13) -> /IORD
- U3 pad 2: /~{IOREQ} -> /IOWR
- U3 pad 3: /~{WR} -> /BDIR
- U3 pad 4: Net-(U3-Pad4) -> /BDIR
- U3 pad 6: /A7 -> Net-(U3-Pad6)
- U3 pad 8: Net-(U3-Pad13) -> unconnected-(U3-Pad8)
- U3 pad 9: Net-(U3-Pad4) -> GND
- U4 pad 10: Net-(U3-Pad1) -> Net-(R2-Pad2)
- U4 pad 11: Net-(U4-Pad11) -> Net-(R1-Pad2)
- U4 pad 13: Net-(R1-Pad2) -> /A1
- U4 pad 3: /A1 -> Net-(U4-Pad12)
- U4 pad 5: /A0 -> Net-(U4-Pad5)
- U4 pad 6: Net-(U4-Pad11) -> /VALID
- U4 pad 8: /BDIR -> Net-(U4-Pad5)
- U4 pad 9: Net-(U4-Pad12) -> Net-(R3-Pad2)
Routing:
- net GND: track 0.00 -> 226.7 mm, vias 0 -> 141
- net VCC: track 0.00 -> 216.2 mm, vias 0 -> 1
- net /~{RESET}: track 0.00 -> 97.0 mm, vias 0 -> 4
- net GND_AUDIO: track 0.00 -> 93.3 mm, vias 0 -> 240
- net /D0: track 0.00 -> 86.8 mm, vias 0 -> 1
- net /D1: track 0.00 -> 80.8 mm, vias 0 -> 2
- net /D7: track 0.00 -> 80.3 mm, vias 0 -> 1
- net /D2: track 0.00 -> 71.7 mm, vias 0 -> 1
- net Net-(CO3-Pin_1): track 0.00 -> 71.5 mm
- net /D3: track 0.00 -> 64.9 mm
- net /A7: track 0.00 -> 61.8 mm, vias 0 -> 1
- net /D6: track 0.00 -> 59.1 mm
- net /D5: track 0.00 -> 59.1 mm
- net Net-(CO3-Pin_2): track 0.00 -> 58.6 mm, vias 0 -> 1
- net /A1: track 0.00 -> 58.5 mm, vias 0 -> 1
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- added copper zone on B.Cu, net GND
- added copper zone on F.Cu, net GND
- added copper zone on B.Cu, net GND_AUDIO
- added copper zone on F.Cu, net GND_AUDIO
Other:
- board text added: "A4"
- board text added: "A5"
- board text added: "A6"
- board text added: "JONZON-X-81 Rev: 1.3 2025 - J.Gratton"
- board text added: "Rev: 1.1 was a change to the Audio Jack connections. Left and Right where connected to Shunts A and B. This also resulted in a Left and Right swap, so Channel A and B where reveresed to compensate."
- board text added: "Rev: 1.2 set Channel A Left (tip), Channel C Right (sleeve) and Chabbel B Mixed."
- board text added: "Rev: 1.3 Corrected Footprints for Logic IC's."
- board text removed: "JONZON-X-81 Rev: 2.0 2025 - J.Gratton"

Commit message: Created rev 1.4 Fab File and Images
Parts:
- added U1A: AY-3-8912, Package_DIP:DIP-28_W15.24mm_LongPads, F.Cu at (100.3, 71.1)
- FB1: renamed from R12; value 0R -> FB
- moved C3 12.0 mm to (95.9, 59.1)
- moved R7 11.1 mm to (76.8, 59.1)
- moved R8 11.1 mm to (71.8, 59.1)
- moved R4 11.1 mm to (92.1, 66.7)
- moved R5 11.1 mm to (87.0, 66.7)
- moved R10 11.1 mm to (61.6, 59.1)
- moved R11 11.1 mm to (56.5, 59.1)
- moved R6 11.1 mm to (81.9, 59.1)
- moved R9 11.1 mm to (66.7, 59.1)
- moved C4 10.5 mm to (95.9, 66.7)
- moved C2 8.84 mm to (55.8, 52.7)
- moved C1 6.62 mm to (65.3, 52.7)
Routing:
- net VCC: track 216.2 -> 268.1 mm, vias 1 -> 0
- net /OUTB: track 18.8 -> 39.4 mm
- net /D2: track 71.7 -> 85.6 mm
- net GND_AUDIO: track 93.3 -> 79.4 mm, vias 240 -> 0
- net /OUTA: track 6.39 -> 18.4 mm
- net /D3: track 64.9 -> 76.9 mm
- net /OUTC: track 21.0 -> 31.5 mm
- net GND: track 226.7 -> 237.0 mm, vias 141 -> 1
- net /D0: track 86.8 -> 96.9 mm
- net /PSGCLK: track 26.4 -> 34.4 mm
- net /CLK: track 52.4 -> 45.2 mm
- net /A1: track 58.5 -> 51.4 mm
- net Net-(R3-Pad2): track 39.0 -> 45.6 mm
- net /~{RESET}: track 97.0 -> 102.7 mm, vias 4 -> 2
- net /D6: track 59.1 -> 64.6 mm
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- removed copper zone on B.Cu, net GND
- removed copper zone on F.Cu, net GND
- removed copper zone on B.Cu, net GND_AUDIO
- removed copper zone on F.Cu, net GND_AUDIO
Other:
- board size 63.5 x 101 mm -> 63.5 x 100.3 mm
- board text added: "JONZON-X-81 Rev: 1.4 2025 - J.Gratton"
- board text added: "Rev: 1.4 Added option for AY-3-8912."
- board text removed: "JONZON-X-81 Rev: 1.3 2025 - J.Gratton"
