File: JONZON-X-81.kicad_sch (KiCad schematic)
At the start: 20 parts, among them SW1 SW_DIP_x01, U1 AY-3-8912, U2 74HCT74, U3 74HCT02, U4 74HCT11

Commit message: rev 1.3
Parts:
- removed SW1: SW_DIP_x01, Button_Switch_SMD:SW_DIP_SPSTx01_Slide_9.78x4.72mm_W8.61mm_P2.54mm, symbol Switch:SW_DIP_x01
- removed U1: AY-3-8912, AY-3-8912:AY-3-8912, symbol AY-3-8912:AY-3-8912
- added C3, C4, C9: 100nf, Capacitor_THT:C_Disc_D3.0mm_W1.6mm_P2.50mm, symbol Device:C_Small
- added CO3: THROUGH, Connector_PinHeader_2.54mm:PinHeader_1x03_P2.54mm_Vertical, symbol Connector_Generic:Conn_01x03
- added R10, R11: 100R, Resistor_THT:R_Axial_DIN0207_L6.3mm_D2.5mm_P7.62mm_Horizontal, symbol Device:R
- added R12: 0R, Resistor_THT:R_Axial_DIN0207_L6.3mm_D2.5mm_P7.62mm_Horizontal, symbol Device:R
- added R2, R3: 47K, Resistor_THT:R_Axial_DIN0207_L6.3mm_D2.5mm_P7.62mm_Horizontal, symbol Device:R
- added SW1: SW_DIP_x03, Button_Switch_THT:SW_DIP_SPSTx03_Slide_9.78x9.8mm_W7.62mm_P2.54mm, symbol Switch:SW_DIP_x03
- added U1: AY-3-8910, Package_DIP:DIP-40_W15.24mm_LongPads, symbol ay-3-8910:AY-3-8910
- added U3: 74HCT08, Package_DIP:DIP-14_W7.62mm_Socket_LongPads, symbol 74xx:74LS08
- R1: value 10K -> 47K
- renumbered C3 to C5, C4 to C6, C5 to C7, C6 to C8, R2 to R4, R3 to R6, R4 to R7, R6 to R8, R7 to R9, U3 to U5
Connections:
- net A0: no longer U4.5
- net A1: now also U4.13; no longer U4.3
- net A4: now also SW1.6
- net A7: now also U3.5; no longer U5.5, U5.6
- net BC1: now also U5.13, U1.29 (BC1); no longer U5.10
- net BDIR: now also U1.27 (BDIR), U3.3, U3.4; no longer U4.8, U5.11, U5.12
- net D0: now also U1.37 (D0)
- net D1: now also U1.36 (D1)
- net D2: now also U1.35 (D2)
- net D3: now also U1.34 (D3)
- net D4: now also U1.33 (D4)
- net D5: now also U1.32 (D5)
- net D6: now also U1.31 (D6)
- net D7: now also U1.30 (D7)
- net GND: now also C9.2, R12.1, U1.1 (GND), U1.24 (A9), U3.10, U3.7 (GND), U3.9; no longer CO2.5, R8.2, R9.2
- net OUTA: now also U1.4 (OUTA)
- net OUTB: now also U1.3 (OUTB)
- net OUTC: now also U1.38 (OUTC)
- net PSGCLK: now also U1.22 (CLOCK)
- net VCC: now also C9.1, R2.1, R3.1, U1.25 (A8), U1.28 (BC2), U1.40 (VCC), U3.14 (VCC)
- net ~{IOREQ}: now also U5.8
- net ~{RESET}: now also U1.23 (RESET)
- net at C2.1, R5.2, R9.1: now also R6.1; no longer R7.1
- net at C2.2: now also R11.1; no longer CO2.4
- net at U4.10: now also R2.2, SW1.2; no longer U5.1
- net at U4.11: now also R1.2, SW1.3; no longer U4.6
- net at U4.9: now also R3.2, SW1.1; no longer U4.12
- net at C1.1, R4.2, R8.1: now also R7.1; no longer R6.1
- net at C1.2: now also R10.1; no longer CO2.1
- net at U5.4: now also U5.11, U5.12; no longer U5.9
- net A6: now reaches CO1.A22 (A6)
- net A6: now also SW1.4
- net A5: now reaches CO1.A23 (A5)
- net A5: now also SW1.5
- net ~{RD}: now reaches CO1.B18 (~{RD})
- net ~{RD}: now also U5.9
- new net: C4.1, CO2.4, CO3.1 (Pin_1), R11.2
- new net: U3.6, U5.5
- new net: U4.5, U4.8
- new net: U3.11, U5.6
- new net: C3.1, CO2.1, CO3.2 (Pin_2), R10.2
- new net: U4.12, U4.3
- new net GND_AUDIO: C3.2, C4.2, CO2.5, CO3.3 (Pin_3), R12.2, R8.2, R9.2
- new net IORD: U3.13, U5.10
- new net IOWR: U3.2, U5.1
- new net VALID: U3.1, U3.12, U4.6
- no-connect marks 36 -> 45
Other:
- note added: "Address Decoding with DIP Switch Options for PSG select addresses of A4,5 and 6 to allow up to 3 PSG's for up to 9 channel sound"
- note added: "Unused Gates"
- note removed: "Address Decoding with DIP Switch Option for ZON X compatibility"
- moved on the sheet: C1, C2, C5, C6, C7, C8, CO2, R1, R4, R5, R6, R7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
