File: JONZON-X-81.kicad_sch (KiCad schematic)
At the start: 31 parts, among them SW1 SW_DIP_x03, U1 AY-3-8910, U1A1 AY-3-8912, U2 74HCT74, U3 74HCT08, U4 74HCT11, U5 74HCT02

Commit message: Created rev 1.4 Fab File and Images
Parts:
- U1A1: footprint (none) -> Package_DIP:DIP-28_W15.24mm_LongPads
Changed lines of the file:
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@@
 			)
 		)
-		(property "Footprint" ""
+		(property "Footprint" "Package_DIP:DIP-28_W15.24mm_LongPads"
 			(at 87.63 248.92 0)
 			(effects
